File: SquareWaveGen.sch (KiCad schematic (older format))
At the start: 26 parts

Commit message: updates
Parts:
- removed Q?: Q_NJFET_DSG, symbol Device:Q_NJFET_DSG
- added U6: LTV-357T, Package_SO:SO-4_4.4x3.6mm_P2.54mm, symbol Isolator:LTV-357T
- C9: renamed from C?; footprint (none) -> Capacitor_SMD:C_0805_2012Metric_Pad1.15x1.40mm_HandSolder
- R14, R15, R16, R17, R18, R19, R20, R21, R22, R23: renamed from R?; footprint (none) -> Resistor_SMD:R_0805_2012Metric_Pad1.15x1.40mm_HandSolder
- gave numbers to parts that had none: 11
Connections:
- wire segments 102 -> 107
