File: ZeroCrossingOctave.sch (KiCad schematic (older format))
At the start: 32 parts

Commit message: updates
Parts:
- added U2: LM2776, Package_TO_SOT_SMD:SOT-23-6, symbol Regulator_SwitchedCapacitor:LM2776
- added U7: LM27762, Package_SON:WSON-12-1EP_3x2mm_P0.5mm_EP1x2.65_ThermalVias, symbol Regulator_SwitchedCapacitor:LM27762
- added U8: LM317_3PinPackage, Package_TO_SOT_SMD:SOT-223-3_TabPin2, symbol Regulator_Linear:LM317_3PinPackage
- C1, C2, C3, C4, C5, C6, C7, C8: renamed from C?; footprint (none) -> Capacitor_SMD:C_0805_2012Metric_Pad1.15x1.40mm_HandSolder
- R1, R10, R11, R12, R13, R2, R3, R4, R5, R6, R7, R8, R9: renamed from R?; footprint (none) -> Resistor_SMD:R_0805_2012Metric_Pad1.15x1.40mm_HandSolder
- gave numbers to parts that had none: 7
Connections:
- wire segments 104 -> 103
